Commit message: update for yaw n slam

File: singbot_description/urdf/singbot.xacro (robot description, xacro)
@@ -122,5 +122,5 @@
 </joint>
 <joint name="Rigid4" type="fixed">
-  <origin xyz="0.0 0.0 0.2" rpy="0 0 0"/>
+  <origin xyz="0.0 0.0 0.2" rpy="0 0 3.14"/>
   <parent link="base_link"/>
   <child link="lidar_1"/>
